File: v2/kicad/kipra-v2/kipra-v2.kicad_pcb (KiCad board)
At the start: 2 copper layers, 159 x 120.6 mm, 47 parts

Commit message: tidy tracks so all F.cu go up interior of MCU
Routing:
- net P2: track 47.4 -> 48.7 mm
- net P19: track 115.6 -> 115.1 mm
